File: file/pcb/body/body.kicad_pcb (KiCad board)
At the start: 2 copper layers, 155.9 x 107.2 mm, 33 parts

Commit message: set the new files
Other:
- outline, holes or cut-outs redrawn
Changed lines of the file:
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@@
     )
     (pad_to_mask_clearance 0)
-    (aux_axis_origin 95.09045 42.680513)
+    (aux_axis_origin 167.351 63.150545)
     (grid_origin 22.69 138.15)
     (pcbplotparams
@@
   (gr_rect (start 84.095 97.463) (end 97.095 107.463)
     (stroke (width 0.15) (type default)) (fill none) (layer "Eco1.User"))
+  (gr_arc (start 87.89145 117.844626) (mid 87.5379 117.698178) (end 87.39145 117.344626)
+    (stroke (width 0.1) (type default)) (layer "Edge.Cuts"))
   (gr_line (start 114.98145 55.824513) (end 114.98145 88.124515)
     (stroke (width 0.1) (type default)) (layer "Edge.Cuts"))
@@
   (gr_arc (start 140.369902 32.560013) (mid 139.052298 33.004542) (end 137.669899 33.155058)
     (stroke (width 0.1) (type default)) (layer "Edge.Cuts"))
+  (gr_line (start 91.39145 117.844626) (end 87.89145 117.844626)
+    (stroke (width 0.1) (type default)) (layer "Edge.Cuts"))
   (gr_arc (start 103.200101 135.570104) (mid 100.26561 136.78561) (end 97.331118 135.570104)
     (stroke (width 0.1) (type default)) (layer "Edge.Cuts"))
   (gr_arc (start 181.169902 31.964513) (mid 179.694507 31.653662) (end 178.469902 30.774013)
     (stroke (width 0.1) (type default)) (layer "Edge.Cuts"))
-  (gr_line (start 108.32445 50.310513) (end 96.09045 50.310513)
+  (gr_line (start 99.05045 52.114513) (end 96.09045 52.114513)
     (stroke (width 0.1) (type default)) (layer "Edge.Cuts"))
   (gr_line (start 194.369902 31.964513) (end 181.169902 31.964513)
@@
   (gr_arc (start 213.869899 41.489968) (mid 215.252294 41.640503) (end 216.569902 42.085013)
     (stroke (width 0.1) (type default)) (layer "Edge.Cuts"))
+  (gr_line (start 103.876388 51.040575) (end 100.538512 51.040575)
+    (stroke (width 0.1) (type default)) (layer "Edge.Cuts"))
+  (gr_arc (start 105.36445 52.114513) (mid 105.17312 52.076433) (end 105.010919 51.968044)
+    (stroke (width 0.1) (type default)) (layer "Edge.Cuts"))
   (gr_line (start 95.09045 42.680513) (end 86.79545 42.680058)
     (stroke (width 0.1) (type default)) (layer "Edge.Cuts"))
@@
   (gr_arc (start 92.43445 91.124515) (mid 90.313121 90.245825) (end 89.43445 88.124515)
     (stroke (width 0.1) (type default)) (layer "Edge.Cuts"))
-  (gr_line (start 91.89145 109.0984) (end 91.89145 116.892626)
+  (gr_line (start 91.89145 108.6464) (end 91.89145 117.344626)
     (stroke (width 0.1) (type default)) (layer "Edge.Cuts"))
   (gr_line (start 162.119902 29.583513) (end 175.769902 29.583513)
@@
   (gr_arc (start 107.707909 131.062297) (mid 122.485033 119.723344) (end 139.693167 112.594849)
     (stroke (width 0.1) (type default)) (layer "Edge.Cuts"))
+  (gr_arc (start 87.39145 108.6464) (mid 87.537897 108.292847) (end 87.89145 108.1464)
+    (stroke (width 0.1) (type default)) (layer "Edge.Cuts"))
   (gr_line (start 152.445104 106.382731) (end 149.26345 94.511918)
     (stroke (width 0.1) (type default)) (layer "Edge.Cuts"))
   (gr_arc (start 97.095 106.963) (mid 96.948553 107.316553) (end 96.595 107.463)
     (stroke (width 0.1) (type default)) (layer "Edge.Cuts"))
+  (gr_line (start 108.32445 52.114513) (end 105.36445 52.114513)
+    (stroke (width 0.1) (type default)) (layer "Edge.Cuts"))
   (gr_line (start 139.693167 112.594849) (end 150.535477 109.689661)
     (stroke (width 0.1) (type default)) (layer "Edge.Cuts"))
+  (gr_arc (start 91.89145 117.344626) (mid 91.745003 117.698179) (end 91.39145 117.844626)
+    (stroke (width 0.1) (type default)) (layer "Edge.Cuts"))
   (gr_line (start 120.319902 37.305511) (end 120.32 39.980998)
     (stroke (width 0.1) (type default)) (layer "Edge.Cuts"))
   (gr_arc (start 84.095 107.963) (mid 84.241447 107.609447) (end 84.595 107.463)
     (stroke (width 0.1) (type default)) (layer "Edge.Cuts"))
-  (gr_line (start 95.59045 49.810513) (end 95.59045 43.180513)
+  (gr_line (start 95.59045 51.614513) (end 95.59045 43.180513)
     (stroke (width 0.1) (type default)) (layer "Edge.Cuts"))
   (gr_arc (start 219.269905 42.680058) (mid 217.887504 42.529543) (end 216.569902 42.085013)
@@
   (gr_line (start 84.095335 121.215729) (end 84.095 107.963)
     (stroke (width 0.1) (type default)) (layer "Edge.Cuts"))
+  (gr_arc (start 103.876388 51.040575) (mid 104.067718 51.078655) (end 104.229919 51.187044)
+    (stroke (width 0.1) (type default)) (layer "Edge.Cuts"))
   (gr_line (start 97.095 97.963) (end 97.095 106.963)
     (stroke (width 0.1) (type default)) (layer "Edge.Cuts"))
-  (gr_arc (start 87.39145 109.0984) (mid 89.64145 108.495514) (end 91.89145 109.0984)
+  (gr_line (start 104.229919 51.187044) (end 105.010919 51.968044)
     (stroke (width 0.1) (type default)) (layer "Edge.Cuts"))
   (gr_line (start 219.269905 101.830058) (end 237.31945 101.830514)
@@
   (gr_arc (start 120.32 39.980998) (mid 119.52906 41.890516) (end 117.619545 42.681453)
     (stroke (width 0.1) (type default)) (layer "Edge.Cuts"))
-  (gr_line (start 87.39145 109.0984) (end 87.39145 116.892626)
-    (stroke (width 0.1) (type default)) (layer "Edge.Cuts"))
-  (gr_line (start 108.824545 43.180998) (end 108.82445 49.810513)
+  (gr_line (start 108.824545 43.180998) (end 108.82445 51.614513)
     (stroke (width 0.1) (type default)) (layer "Edge.Cuts"))
   (gr_arc (start 200.6699 100.639513) (mid 198.131592 99.790256) (end 196.615352 97.584513)
@@
   (gr_arc (start 108.824545 43.180998) (mid 108.970992 42.827445) (end 109.324545 42.680998)
     (stroke (width 0.1) (type default)) (layer "Edge.Cuts"))
+  (gr_line (start 87.39145 108.6464) (end 87.39145 117.344626)
+    (stroke (width 0.1) (type default)) (layer "Edge.Cuts"))
   (gr_arc (start 219.269905 101.830058) (mid 217.88751 101.679524) (end 216.569902 101.235013)
     (stroke (width 0.1) (type default)) (layer "Edge.Cuts"))
@@
   (gr_arc (start 84.094995 45.380513) (mid 84.88594 43.471003) (end 86.79545 42.680058)
     (stroke (width 0.1) (type default)) (layer "Edge.Cuts"))
+  (gr_line (start 87.89145 108.1464) (end 91.39145 108.1464)
+    (stroke (width 0.1) (type default)) (layer "Edge.Cuts"))
   (gr_line (start 137.669899 33.155058) (end 124.4699 33.155513)
     (stroke (width 0.1) (type default)) (layer "Edge.Cuts"))
@@
   (gr_arc (start 120.319902 37.305511) (mid 121.535406 34.371003) (end 124.4699 33.155513)
     (stroke (width 0.1) (type default)) (layer "Edge.Cuts"))
-  (gr_arc (start 96.09045 50.310513) (mid 95.736897 50.164066) (end 95.59045 49.810513)
+  (gr_arc (start 96.09045 52.114513) (mid 95.736924 51.96805) (end 95.59045 51.614513)
     (stroke (width 0.1) (type default)) (layer "Edge.Cuts"))
   (gr_line (start 84.094995 45.380513) (end 84.095 96.963)
     (stroke (width 0.1) (type default)) (layer "Edge.Cuts"))
-  (gr_arc (start 108.82445 49.810513) (mid 108.678003 50.164066) (end 108.32445 50.310513)
+  (gr_arc (start 108.82445 51.614513) (mid 108.678002 51.968076) (end 108.32445 52.114513)
+    (stroke (width 0.1) (type default)) (layer "Edge.Cuts"))
+  (gr_arc (start 99.403981 51.968044) (mid 99.24178 52.076433) (end 99.05045 52.114513)
     (stroke (width 0.1) (type default)) (layer "Edge.Cuts"))
   (gr_line (start 103.200101 135.570104) (end 107.707909 131.062297)
     (stroke (width 0.1) (type default)) (layer "Edge.Cuts"))
-  (gr_arc (start 91.89145 116.892626) (mid 89.64145 117.495512) (end 87.39145 116.892626)
+  (gr_arc (start 100.184981 51.187044) (mid 100.347182 51.078655) (end 100.538512 51.040575)
+    (stroke (width 0.1) (type default)) (layer "Edge.Cuts"))
+  (gr_line (start 100.184981 51.187044) (end 99.403981 51.968044)
     (stroke (width 0.1) (type default)) (layer "Edge.Cuts"))
   (gr_arc (start 111.98145 52.824513) (mid 114.102798 53.703176) (end 114.98145 55.824513)
@@
   (gr_line (start 213.869899 100.639968) (end 200.6699 100.639513)
     (stroke (width 0.1) (type default)) (layer "Edge.Cuts"))
+  (gr_arc (start 91.39145 108.1464) (mid 91.745003 108.292847) (end 91.89145 108.6464)
+    (stroke (width 0.1) (type default)) (layer "Edge.Cuts"))
   (gr_arc (start 84.886146 123.124917) (mid 84.300858 122.248974) (end 84.095335 121.215729)
     (stroke (width 0.1) (type default)) (layer "Edge.Cuts"))
   (gr_line (start 92.43445 91.124515) (end 111.98145 91.124515)
     (stroke (width 0.1) (type default)) (layer "Edge.Cuts"))
+  (gr_rect (start 105.520334 50.310513) (end 108.480334 51.770513)
+    (stroke (width 0.05) (type default)) (fill none) (layer "F.CrtYd"))
+  (gr_rect (start 95.940334 50.310513) (end 98.900334 51.770513)
+    (stroke (width 0.05) (type default)) (fill none) (layer "F.CrtYd"))
   (gr_text "Thickness: 1.6mm" (at 84.14 36.1) (layer "Eco2.User")
     (effects (font (size 2 2) (thickness 0.15)) (justify left bottom))
