File: file/pcb/main/main.kicad_pcb (KiCad board)
At the start: 2 copper layers, 155.9 x 107.2 mm, 68 parts, among them J1 AudioJack3, J2 TPS43-201A-S, J3 TPS43-201A-S, K1 PG1316S, K10 PG1316S, K11 PG1316S, K12 PG1316S, K13 PG1316S, K14 PG1316S, K15 PG1316S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

Commit message: set the new files
Parts:
- added L5: SK6805, DreaM117er-keebLibrary:LED_SK6805_PLCC4_2.4x2.7mm_P1.3mm, F.Cu at (170.2, 136.4)
- added L6: SK6805, DreaM117er-keebLibrary:LED_SK6805_PLCC4_2.4x2.7mm_P1.3mm, B.Cu at (170.2, 136.4)
- added R1: 5.1K, Resistor_SMD:R_0603_1608Metric, F.Cu at (187.6, 71.5)
- added R2: 5.1K, Resistor_SMD:R_0603_1608Metric, F.Cu at (178.0, 71.5)
- added R3: 5.1K, Resistor_SMD:R_0603_1608Metric, B.Cu at (187.6, 71.5)
- added R4: 5.1K, Resistor_SMD:R_0603_1608Metric, B.Cu at (178.0, 71.5)
- K1, K10, K11, K12, K13, K14, K15, K16, K17, K18, K19, K2, K20, K21, K3, K4, K5, K6, K7, K8, K9: footprint DreaM117er-keebLibrary:SW_Kailh_PG1316S_1.00u_Dual -> DreaM117er-keebLibrary:SW_Kailh_PG1316S_1.00u_Dual2
- moved L2 2.43 mm to (170.2, 133.5), turned to 0 degrees
- moved L4 2.43 mm to (170.2, 133.5), turned to 0 degrees
- moved L1 0.34 mm to (170.2, 130.6), turned to 0 degrees
- moved L3 0.34 mm to (170.2, 130.6), turned to 0 degrees
Connections:
- J1 pad T: +3V3 -> +5V
- L2 pad 1: unconnected-(L2-DOUT-Pad1) -> Net-(L2-DOUT)
- L4 pad 1: unconnected-(L4-DOUT-Pad1) -> Net-(L2-DOUT)
- P1 pad A5: unconnected-(P1-CC1-PadA5) -> Net-(P1-CC1)
- P1 pad B5: unconnected-(P1-CC2-PadB5) -> Net-(P1-CC2)
- P2 pad A5: unconnected-(P2-CC1-PadA5) -> Net-(P1-CC2)
- P2 pad B5: unconnected-(P2-CC2-PadB5) -> Net-(P1-CC1)
Routing:
- net +3V3: track 103.7 -> 74.2 mm, vias 4 -> 2
- net +5V: track 142.4 -> 116.1 mm, vias 9 -> 11
- net GND: track 80.3 -> 106.4 mm, vias 4 -> 3
- net Net-(L2-DOUT): track 0.00 -> 10.0 mm, vias 0 -> 2
- net Net-(P1-CC2): track 0.00 -> 6.02 mm, vias 0 -> 2
- net Net-(P1-CC1): track 0.00 -> 6.01 mm, vias 0 -> 2
- net Net-(L1-DOUT): track 7.08 -> 10.0 mm, vias 1 -> 2
- net RGB: track 57.1 -> 55.5 mm
