File: file/pcb/main/main.kicad_sch (KiCad schematic)
At the start: 66 parts, among them J1 AudioJack3, J2 TPS43-201A-S, J3 TPS43-201A-S, K1 PG1316S, K10 PG1316S, K11 PG1316S, K12 PG1316S, K13 PG1316S, K14 PG1316S, K15 PG1316S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

Commit message: set the new files
Parts:
- added L5, L6: SK6805, DreaM117er-keebLibrary:LED_SK6805_PLCC4_2.4x2.7mm_P1.3mm, symbol LED:SK6805
- added R1, R2, R3, R4: 5.1K, Resistor_SMD:R_0603_1608Metric, symbol Device:R
- K1, K10, K11, K12, K13, K14, K15, K16, K17, K18, K19, K2, K20, K21, K3, K4, K5, K6, K7, K8, K9: footprint DreaM117er-keebLibrary:SW_Kailh_PG1316S_1.00u_Dual -> DreaM117er-keebLibrary:SW_Kailh_PG1316S_1.00u_Dual2
Connections:
- net +3V3: no longer J1.T
- net +5V: now also J1.T, L5.4 (VDD), L6.4 (VDD)
- net GND: now also L5.2 (VSS), L6.2 (VSS), R1.2, R2.2, R3.2, R4.2
- net at P1.A5 (CC1): now also P2.B5 (CC2), R1.1, R3.1
- net at P1.B5 (CC2): now also P2.A5 (CC1), R2.1, R4.1
- net at L2.1 (DOUT): now also L4.1 (DOUT), L5.3 (DIN), L6.3 (DIN)
- no-connect marks 26 -> 22
Other:
- moved on the sheet: P2
